Commit message: Add support to load stl

File: configs/urdfs/myohand_kinematics_hand_only_axis_aligned.urdf (robot description, URDF)
Before this commit: robot converted_robot, 38 links, 37 joints
Links:
- link capitate: geometry visual mesh filename=file:///home/haochen/catkin_ws/src/relaxed_ik_ros1/relaxed_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
- link distal_thumb: geometry visual mesh filename=file:///home/haochen/catkin_ws/src/relaxed_ik_ros1/relaxed_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
- link distph2: geometry visual mesh filename=file:///home/haochen/catkin_ws/src/relaxed_ik_ros1/relaxed_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
- link distph3: geometry visual mesh filename=file:///home/haochen/catkin_ws/src/relaxed_ik_ros1/relaxed_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
- link distph4: geometry visual mesh filename=file:///home/haochen/catkin_ws/src/relaxed_ik_ros1/relaxed_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
- link distph5: geometry visual mesh filename=file:///home/haochen/catkin_ws/src/relaxed_ik_ros1/relaxed_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
- link fifthmc: geometry visual mesh filename=file:///home/haochen/catkin_ws/src/relaxed_ik_ros1/relaxed_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
- link firstmc: geometry visual mesh filename=file:///home/haochen/catkin_ws/src/relaxed_ik_ros1/relaxed_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
- link fourthmc: geometry visual mesh filename=file:///home/haochen/catkin_ws/src/relaxed_ik_ros1/relaxed_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
- link hamate: geometry visual mesh filename=file:///home/haochen/catkin_ws/src/relaxed_ik_ros1/relaxed_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
- link lunate: geometry visual mesh filename=file:///home/haochen/catkin_ws/src/relaxed_ik_ros1/relaxed_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
- link midph2: geometry visual mesh filename=file:///home/haochen/catkin_ws/src/relaxed_ik_ros1/relaxed_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
- link midph3: geometry visual mesh filename=file:///home/haochen/catkin_ws/src/relaxed_ik_ros1/relaxed_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
- link midph4: geometry visual mesh filename=file:///home/haochen/catkin_ws/src/relaxed_ik_ros1/relaxed_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
- link midph5: geometry visual mesh filename=file:///home/haochen/catkin_ws/src/relaxed_ik_ros1/relaxed_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
- link pisiform: geometry visual mesh filename=file:///home/haochen/catkin_ws/src/relaxed_ik_ros1/relaxed_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
- link proximal_thumb: geometry visual mesh filename=file:///home/haochen/catkin_ws/src/relaxed_ik_ros1/relaxed_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
- link proxph2: geometry visual mesh filename=file:///home/haochen/catkin_ws/src/relaxed_ik_ros1/relaxed_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
- link proxph3: geometry visual mesh filename=file:///home/haochen/catkin_ws/src/relaxed_ik_ros1/relaxed_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
- link proxph4: geometry visual mesh filename=file:///home/haochen/catkin_ws/src/relaxed_ik_ros1/relaxed_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
- link proxph5: geometry visual mesh filename=file:///home/haochen/catkin_ws/src/relaxed_ik_ros1/relaxed_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
- link scaphoid: geometry visual mesh filename=file:///home/haochen/catkin_ws/src/relaxed_ik_ros1/relaxed_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
- link secondmc: geometry visual mesh filename=file:///home/haochen/catkin_ws/src/relaxed_ik_ros1/relaxed_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
- link thirdmc: geometry visual mesh filename=file:///home/haochen/catkin_ws/src/relaxed_ik_ros1/relaxed_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
- link trapezium: geometry visual mesh filename=file:///home/haochen/catkin_ws/src/relaxed_ik_ros1/relaxed_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
- link trapezoid: geometry visual mesh filename=file:///home/haochen/catkin_ws/src/relaxed_ik_ros1/relaxed_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
- link triquetrum: geometry visual mesh filename=file:///home/haochen/catkin_ws/src/relaxed_ik_ros1/relaxed_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
- link world: mass 0.0 -> None
Joints:
- removed joint floating_joint
- added joint fixed_joint: type fixed, parent world, child lunate, origin xyz=0 0 0 rpy=0 0 0

Commit message: Update the base of the myohand

File: configs/urdfs/myohand_kinematics_hand_only_axis_aligned.urdf (robot description, URDF)
Before this commit: robot converted_robot, 38 links, 37 joints
Links:
- added link joint_rx_link
- added link joint_ry_link
- added link joint_rz_link
- added link joint_tx_link
- added link joint_ty_link
- added link joint_tz_link
Joints:
- removed joint fixed_joint
- added joint rotate_x_joint: type revolute, parent joint_tz_link, child joint_rx_link, origin xyz=0 0 0 rpy=0 0 0, axis 1 0 0, limit lower=-3.141593 upper=3.141593 effort=100 velocity=100
- added joint rotate_y_joint: type revolute, parent joint_rx_link, child joint_ry_link, origin xyz=0 0 0 rpy=0 0 0, axis 0 1 0, limit lower=-3.141593 upper=3.141593 effort=100 velocity=100
- added joint rotate_z_joint: type revolute, parent joint_ry_link, child joint_rz_link, origin xyz=0 0 0 rpy=0 0 0, axis 0 0 1, limit lower=-3.141593 upper=3.141593 effort=100 velocity=100
- added joint translate_x_joint: type prismatic, parent world, child joint_tx_link, origin xyz=0 0 0 rpy=0 0 0, axis 1 0 0, limit lower=-1.0 upper=1.0 effort=20.0 velocity=5.0
- added joint translate_y_joint: type prismatic, parent joint_tx_link, child joint_ty_link, origin xyz=0 0 0 rpy=0 0 0, axis 0 1 0, limit lower=-1.0 upper=1.0 effort=20.0 velocity=5.0
- added joint translate_z_joint: type prismatic, parent joint_ty_link, child joint_tz_link, origin xyz=0 0 0 rpy=0 0 0, axis 0 0 1, limit lower=-1.0 upper=1.0 effort=20.0 velocity=5.0
- added joint wrist_fixed: type fixed, parent joint_rz_link, child lunate, origin xyz=0 0 0 rpy=0 0 0
