Commit message: Add two hands to the urdf

File: configs/urdfs/myohand_kinematics_hand_only_axis_aligned.urdf (robot description, URDF)
Before this commit: robot converted_robot, 44 links, 43 joints
Links:
- added link IFtip_left, mass 0.001
- added link LFtip_left, mass 0.001
- added link MFtip_left, mass 0.001
- added link RFtip_left, mass 0.001
- added link THtip_left, mass 0.001
- added link capitate_left, mass 0.001912230829037991; visual mesh filename=file:///home/haochen/catkin_ws/src/relaxed_ik_ros1/relaxed_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 scale=1.1486480425226826 1.1486480425226826 1.1486480425226826
- added link cmc_abduction_dummy_left, mass 0.001
- added link distal_thumb_left, mass 0.003; visual mesh filename=file:///home/haochen/catkin_ws/src/relaxed_ik_ros1/relaxed_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 scale=1.1486480425226826 1.1486480425226826 1.1486480425226826
- added link distph2_left, mass 0.002; visual mesh filename=file:///home/haochen/catkin_ws/src/relaxed_ik_ros1/relaxed_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 scale=1.1486480425226826 1.1486480425226826 1.1486480425226826
- added link distph3_left, mass 0.002; visual mesh filename=file:///home/haochen/catkin_ws/src/relaxed_ik_ros1/relaxed_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 scale=1.1486480425226826 1.1486480425226826 1.1486480425226826
- added link distph4_left, mass 0.002; visual mesh filename=file:///home/haochen/catkin_ws/src/relaxed_ik_ros1/relaxed_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 scale=1.1486480425226826 1.1486480425226826 1.1486480425226826
- added link distph5_left, mass 0.001; visual mesh filename=file:///home/haochen/catkin_ws/src/relaxed_ik_ros1/relaxed_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 scale=1.1486480425226826 1.1486480425226826 1.1486480425226826
- added link fifthmc_left, mass 0.02; visual mesh filename=file:///home/haochen/catkin_ws/src/relaxed_ik_ros1/relaxed_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 scale=1.1486480425226826 1.1486480425226826 1.1486480425226826
- added link firstmc_left, mass 0.016; visual mesh filename=file:///home/haochen/catkin_ws/src/relaxed_ik_ros1/relaxed_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 scale=1.1486480425226826 1.1486480425226826 1.1486480425226826
- added link fourthmc_left, mass 0.02; visual mesh filename=file:///home/haochen/catkin_ws/src/relaxed_ik_ros1/relaxed_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 scale=1.1486480425226826 1.1486480425226826 1.1486480425226826
- added link hamate_left, mass 0.02; visual mesh filename=file:///home/haochen/catkin_ws/src/relaxed_ik_ros1/relaxed_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 scale=1.1486480425226826 1.1486480425226826 1.1486480425226826
- added link joint_rx_link_left
- added link joint_ry_link_left
- added link joint_rz_link_left
- added link joint_tx_link_left
- added link joint_ty_link_left
- added link joint_tz_link_left
- added link lunate_left, mass 0.0012000263535597198; visual mesh filename=file:///home/haochen/catkin_ws/src/relaxed_ik_ros1/relaxed_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 scale=1.1486480425226826 1.1486480425226826 1.1486480425226826
- added link mcp2_flexion_dummy_left, mass 0.001
- added link mcp3_flexion_dummy_left, mass 0.001
- added link mcp4_flexion_dummy_left, mass 0.001
- added link mcp5_flexion_dummy_left, mass 0.001
- added link midph2_left, mass 0.003; visual mesh filename=file:///home/haochen/catkin_ws/src/relaxed_ik_ros1/relaxed_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 scale=1.1486480425226826 1.1486480425226826 1.1486480425226826
- added link midph3_left, mass 0.002; visual mesh filename=file:///home/haochen/catkin_ws/src/relaxed_ik_ros1/relaxed_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 scale=1.1486480425226826 1.1486480425226826 1.1486480425226826
- added link midph4_left, mass 0.003; visual mesh filename=file:///home/haochen/catkin_ws/src/relaxed_ik_ros1/relaxed_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 scale=1.1486480425226826 1.1486480425226826 1.1486480425226826
- added link midph5_left, mass 0.002; visual mesh filename=file:///home/haochen/catkin_ws/src/relaxed_ik_ros1/relaxed_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 scale=1.1486480425226826 1.1486480425226826 1.1486480425226826
- added link pisiform_left, mass 0.02; visual mesh filename=file:///home/haochen/catkin_ws/src/relaxed_ik_ros1/relaxed_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 scale=1.1486480425226826 1.1486480425226826 1.1486480425226826
- added link proximal_thumb_left, mass 0.0079; visual mesh filename=file:///home/haochen/catkin_ws/src/relaxed_ik_ros1/relaxed_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 scale=1.1486480425226826 1.1486480425226826 1.1486480425226826
- added link proxph2_left, mass 0.01; visual mesh filename=file:///home/haochen/catkin_ws/src/relaxed_ik_ros1/relaxed_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 scale=1.1486480425226826 1.1486480425226826 1.1486480425226826
- added link proxph3_left, mass 0.01; visual mesh filename=file:///home/haochen/catkin_ws/src/relaxed_ik_ros1/relaxed_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 scale=1.1486480425226826 1.1486480425226826 1.1486480425226826
- added link proxph4_left, mass 0.01; visual mesh filename=file:///home/haochen/catkin_ws/src/relaxed_ik_ros1/relaxed_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 scale=1.1486480425226826 1.1486480425226826 1.1486480425226826
- added link proxph5_left, mass 0.005; visual mesh filename=file:///home/haochen/catkin_ws/src/relaxed_ik_ros1/relaxed_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 scale=1.1486480425226826 1.1486480425226826 1.1486480425226826
- added link scaphoid_left, mass 0.02; visual mesh filename=file:///home/haochen/catkin_ws/src/relaxed_ik_ros1/relaxed_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 scale=1.1486480425226826 1.1486480425226826 1.1486480425226826
- added link secondmc_left, mass 0.02; visual mesh filename=file:///home/haochen/catkin_ws/src/relaxed_ik_ros1/relaxed_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 scale=1.1486480425226826 1.1486480425226826 1.1486480425226826
- added link thirdmc_left, mass 0.02; visual mesh filename=file:///home/haochen/catkin_ws/src/relaxed_ik_ros1/relaxed_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 scale=1.1486480425226826 1.1486480425226826 1.1486480425226826
- added link trapezium_left, mass 0.02; visual mesh filename=file:///home/haochen/catkin_ws/src/relaxed_ik_ros1/relaxed_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 scale=1.1486480425226826 1.1486480425226826 1.1486480425226826
- added link trapezoid_left, mass 0.02; visual mesh filename=file:///home/haochen/catkin_ws/src/relaxed_ik_ros1/relaxed_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 scale=1.1486480425226826 1.1486480425226826 1.1486480425226826
- added link triquetrum_left, mass 0.02; visual mesh filename=file:///home/haochen/catkin_ws/src/relaxed_ik_ros1/relaxed_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 scale=1.1486480425226826 1.1486480425226826 1.1486480425226826
- link capitate: geometry visual mesh filename=file:///home/haochen/catkin_ws/src/relaxed_ik_ros1/relaxed_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 scale=1.1486480425226826 1.1486480425226826 1.1486480425226826
- link distal_thumb: geometry visual mesh filename=file:///home/haochen/catkin_ws/src/relaxed_ik_ros1/relaxed_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 scale=1.1486480425226826 1.1486480425226826 1.1486480425226826
- link distph2: geometry visual mesh filename=file:///home/haochen/catkin_ws/src/relaxed_ik_ros1/relaxed_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 scale=1.1486480425226826 1.1486480425226826 1.1486480425226826
- link distph3: geometry visual mesh filename=file:///home/haochen/catkin_ws/src/relaxed_ik_ros1/relaxed_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 scale=1.1486480425226826 1.1486480425226826 1.1486480425226826
- link distph4: geometry visual mesh filename=file:///home/haochen/catkin_ws/src/relaxed_ik_ros1/relaxed_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 scale=1.1486480425226826 1.1486480425226826 1.1486480425226826
- link distph5: geometry visual mesh filename=file:///home/haochen/catkin_ws/src/relaxed_ik_ros1/relaxed_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 scale=1.1486480425226826 1.1486480425226826 1.1486480425226826
- link fifthmc: geometry visual mesh filename=file:///home/haochen/catkin_ws/src/relaxed_ik_ros1/relaxed_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 scale=1.1486480425226826 1.1486480425226826 1.1486480425226826
- link firstmc: geometry visual mesh filename=file:///home/haochen/catkin_ws/src/relaxed_ik_ros1/relaxed_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 scale=1.1486480425226826 1.1486480425226826 1.1486480425226826
- link fourthmc: geometry visual mesh filename=file:///home/haochen/catkin_ws/src/relaxed_ik_ros1/relaxed_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 scale=1.1486480425226826 1.1486480425226826 1.1486480425226826
- link hamate: geometry visual mesh filename=file:///home/haochen/catkin_ws/src/relaxed_ik_ros1/relaxed_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 scale=1.1486480425226826 1.1486480425226826 1.1486480425226826
- link lunate: geometry visual mesh filename=file:///home/haochen/catkin_ws/src/relaxed_ik_ros1/relaxed_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 scale=1.1486480425226826 1.1486480425226826 1.1486480425226826
- link midph2: geometry visual mesh filename=file:///home/haochen/catkin_ws/src/relaxed_ik_ros1/relaxed_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 scale=1.1486480425226826 1.1486480425226826 1.1486480425226826
- link midph3: geometry visual mesh filename=file:///home/haochen/catkin_ws/src/relaxed_ik_ros1/relaxed_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 scale=1.1486480425226826 1.1486480425226826 1.1486480425226826
- link midph4: geometry visual mesh filename=file:///home/haochen/catkin_ws/src/relaxed_ik_ros1/relaxed_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 scale=1.1486480425226826 1.1486480425226826 1.1486480425226826
- link midph5: geometry visual mesh filename=file:///home/haochen/catkin_ws/src/relaxed_ik_ros1/relaxed_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 scale=1.1486480425226826 1.1486480425226826 1.1486480425226826
- link pisiform: geometry visual mesh filename=file:///home/haochen/catkin_ws/src/relaxed_ik_ros1/relaxed_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 scale=1.1486480425226826 1.1486480425226826 1.1486480425226826
- link proximal_thumb: geometry visual mesh filename=file:///home/haochen/catkin_ws/src/relaxed_ik_ros1/relaxed_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 scale=1.1486480425226826 1.1486480425226826 1.1486480425226826
- link proxph2: geometry visual mesh filename=file:///home/haochen/catkin_ws/src/relaxed_ik_ros1/relaxed_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 scale=1.1486480425226826 1.1486480425226826 1.1486480425226826
- link proxph3: geometry visual mesh filename=file:///home/haochen/catkin_ws/src/relaxed_ik_ros1/relaxed_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 scale=1.1486480425226826 1.1486480425226826 1.1486480425226826
- link proxph4: geometry visual mesh filename=file:///home/haochen/catkin_ws/src/relaxed_ik_ros1/relaxed_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 scale=1.1486480425226826 1.1486480425226826 1.1486480425226826
- link proxph5: geometry visual mesh filename=file:///home/haochen/catkin_ws/src/relaxed_ik_ros1/relaxed_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 scale=1.1486480425226826 1.1486480425226826 1.1486480425226826
- link scaphoid: geometry visual mesh filename=file:///home/haochen/catkin_ws/src/relaxed_ik_ros1/relaxed_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 scale=1.1486480425226826 1.1486480425226826 1.1486480425226826
- link secondmc: geometry visual mesh filename=file:///home/haochen/catkin_ws/src/relaxed_ik_ros1/relaxed_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 scale=1.1486480425226826 1.1486480425226826 1.1486480425226826
- link thirdmc: geometry visual mesh filename=file:///home/haochen/catkin_ws/src/relaxed_ik_ros1/relaxed_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 scale=1.1486480425226826 1.1486480425226826 1.1486480425226826
- link trapezium: geometry visual mesh filename=file:///home/haochen/catkin_ws/src/relaxed_ik_ros1/relaxed_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 scale=1.1486480425226826 1.1486480425226826 1.1486480425226826
- link trapezoid: geometry visual mesh filename=file:///home/haochen/catkin_ws/src/relaxed_ik_ros1/relaxed_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 scale=1.1486480425226826 1.1486480425226826 1.1486480425226826
- link triquetrum: geometry visual mesh filename=file:///home/haochen/catkin_ws/src/relaxed_ik_ros1/relaxed_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 scale=1.1486480425226826 1.1486480425226826 1.1486480425226826
Joints:
- added joint IFtip_joint_left: type fixed, parent distph2_left, child IFtip_left, origin xyz=-0.002076706726373289 -0.020697797526362027 0.00022169691984058083 rpy=1.5707963267948983 1.4707963268582902 1.4707963268582915
- added joint LFtip_joint_left: type fixed, parent distph5_left, child LFtip_left, origin xyz=0.0003031599163330718 -0.01982519198469429 0.0011696846527624316 rpy=-0.30068756862856233 0.6985554313998295 -0.11023436132302195
- added joint MFtip_joint_left: type fixed, parent distph3_left, child MFtip_left, origin xyz=-0.0022972960850453656 -0.021824312807930957 -0.001148648042522682 rpy=0.0 0.0 0.0
- added joint RFtip_joint_left: type fixed, parent distph4_left, child RFtip_left, origin xyz=0.0015965954281736243 -0.020675664765408275 -0.0002994456376664131 rpy=9.507900496666728e-34 0.9707969349430008 -3.875608070853002e-33
- added joint THtip_joint_left: type fixed, parent distal_thumb_left, child THtip_left, origin xyz=-0.011304973256230644 -0.02471051649524722 0.0023927444174953946 rpy=-0.5009125402511723 -0.05012299056598346 0.012825373716091937
- added joint capitate2fifthmc_fixed_left: type fixed, parent capitate_left, child fifthmc_left, origin xyz=0.025150797539076657 -0.0398385600588142 -0.004844997443360676 rpy=0.0 0.0 0.0
- added joint capitate2fourthmc_fixed_left: type fixed, parent capitate_left, child fourthmc_left, origin xyz=0.013836614320228233 -0.04654207003497658 0.004035200573382184 rpy=0.0 0.0 0.0
- added joint capitate2hamate_fixed_left: type fixed, parent capitate_left, child hamate_left, origin xyz=0.012599520378431307 -0.002865876866094092 -0.0008614860318920119 rpy=0.0 0.0 0.0
- added joint capitate2secondmc_fixed_left: type fixed, parent capitate_left, child secondmc_left, origin xyz=-0.016867896504445593 -0.04321213935970332 0.00577999694997414 rpy=0.0 0.0 0.0
- added joint capitate2thirdmc_fixed_left: type fixed, parent capitate_left, child thirdmc_left, origin xyz=-0.0005479051162833194 -0.045071800540547546 0.00847357660968983 rpy=0.0 0.0 0.0
- added joint capitate2trapezium_fixed_left: type fixed, parent capitate_left, child trapezium_left, origin xyz=-0.017566274514299384 -0.005248172906286139 -0.01184026402232381 rpy=0.0 0.0 0.0
- added joint capitate2trapezoid_fixed_left: type fixed, parent capitate_left, child trapezoid_left, origin xyz=-0.010502089052784887 -0.004665808348727138 -0.00283026877677589 rpy=0.0 0.0 0.0
- added joint cmc_abduction_left: type revolute, parent trapezium_left, child cmc_abduction_dummy_left, origin xyz=-0.008270265906163317 -0.006202699429622488 -0.002871620106306705 rpy=0.7286789533902661 0.04241170412851947 0.01617642349516324, axis 1.747988441681546e-18 -1.0772761261336016e-16 -1.0, limit lower=-0.5 upper=0.78 effort=100 velocity=100
- added joint cmc_flexion_left: type revolute, parent cmc_abduction_dummy_left, child firstmc_left, origin xyz=-6.938893903907228e-18 -6.938893903907228e-18 1.214306433183765e-17 rpy=-1.7353556432102097 -0.24272282231633158 0.5745472836968706, axis -2.8391311673900116e-17 -5.045193471461809e-17 -1.0000000000000002, limit lower=-0.78 upper=0.7 effort=100 velocity=100
- added joint ip_flexion_left: type revolute, parent proximal_thumb_left, child distal_thumb_left, origin xyz=-0.01530361676331593 -0.03162676148079482 -0.0066182282430972406 rpy=0.29479434175333596 -0.03270997999703473 0.011022901491355958, axis -1.923774407218676e-17 -2.7135002682840594e-16 -1.0000000000000009, limit lower=-1.309 upper=0.436332 effort=100 velocity=100
- added joint lunate2capitate_fixed_left: type fixed, parent lunate_left, child capitate_left, origin xyz=-0.004585402985750549 -0.017291747632136464 0.0026729039949502827 rpy=0.0 0.0 0.0
- added joint lunate2pisiform_fixed_left: type fixed, parent lunate_left, child pisiform_left, origin xyz=0.015378099993293676 -0.011355534548379242 -0.012167628714442777 rpy=0.0 0.0 0.0
- added joint lunate2scaphoid_fixed_left: type fixed, parent lunate_left, child scaphoid_left, origin xyz=-0.014180060084942516 -0.005127564861821255 -0.001440404645323444 rpy=0.0 0.0 0.0
- added joint lunate2triquetrum_fixed_left: type fixed, parent lunate_left, child triquetrum_left, origin xyz=0.01238702049056461 -0.008613711670877596 -0.001480607326811738 rpy=0.0 0.0 0.0
- added joint mcp2_abduction_left: type revolute, parent mcp2_flexion_dummy_left, child proxph2_left, origin xyz=6.938893903907228e-18 2.7755575615628914e-17 5.204170427930421e-18 rpy=1.996706135703523 1.4588445662369582 1.9856122470713673, axis -2.8382323702885056e-16 2.4019512150402412e-17 -0.9999999999999999, limit lower=-0.261799 upper=0.261799 effort=100 velocity=100
- added joint mcp2_flexion_left: type revolute, parent secondmc_left, child mcp2_flexion_dummy_left, origin xyz=-0.004021416796871912 -0.032441266664968126 0.004158105913932111 rpy=-1.5707963267948977 -1.4708802086674053 1.4708802086674064, axis -5.2438525824824176e-20 7.039945989835385e-18 -1.0, limit lower=0.0 upper=1.5708 effort=100 velocity=100
- added joint mcp3_abduction_left: type revolute, parent mcp3_flexion_dummy_left, child proxph3_left, origin xyz=3.2526065174565133e-19 -1.3877787807814457e-17 0.0 rpy=-0.0 1.5707963267948961 0.0, axis -4.59135596783022e-18 0.0 -1.0, limit lower=-0.261799 upper=0.261799 effort=100 velocity=100
- added joint mcp3_flexion_left: type revolute, parent thirdmc_left, child mcp3_flexion_dummy_left, origin xyz=-0.0002756755302054433 -0.03019795703792133 0.00204229621960533 rpy=0.0 -1.370796734865936 0.0, axis 1.842288986358278e-17 0.0 -1.0, limit lower=0.0 upper=1.5708 effort=100 velocity=100
- added joint mcp4_abduction_left: type revolute, parent mcp4_flexion_dummy_left, child proxph4_left, origin xyz=3.469446951953614e-18 -1.3877787807814457e-17 1.6263032587282567e-19 rpy=-0.0 1.5707963267948961 0.0, axis 4.994681042330142e-17 0.0 -1.0000000000000002, limit lower=-0.261799 upper=0.261799 effort=100 velocity=100
- added joint mcp4_flexion_left: type revolute, parent fourthmc_left, child mcp4_flexion_dummy_left, origin xyz=0.002102025917816509 -0.02721032347931983 -0.0001987161113564239 rpy=0.0 -1.1207958627668684 0.0, axis -7.907580905939781e-17 0.0 -1.0, limit lower=0.0 upper=1.5708 effort=100 velocity=100
- added joint mcp5_abduction_left: type revolute, parent mcp5_flexion_dummy_left, child proxph5_left, origin xyz=3.469446951953614e-18 0.0 -1.734723475976807e-18 rpy=-0.0 1.5707963267948966 0.0, axis 1.804436795852415e-16 0.0 -1.0000000000000002, limit lower=-0.261799 upper=0.261799 effort=100 velocity=100
- added joint mcp5_flexion_left: type revolute, parent fifthmc_left, child mcp5_flexion_dummy_left, origin xyz=0.0018343909239087238 -0.024616676199303605 -0.0017183774716139338 rpy=0.0 -0.9707969349430003 0.0, axis 2.7011479700438378e-17 0.0 -1.0, limit lower=0.0 upper=1.5708 effort=100 velocity=100
- added joint md2_flexion_left: type revolute, parent midph2_left, child distph2_left, origin xyz=-0.0013930466537968242 -0.028836877205181244 0.0006023764869396448 rpy=0.022138329695812073 0.19777869365516998 -2.5098334244374673e-05, axis -2.4455606779405633e-18 -4.090344666757575e-17 -0.9999999999999998, limit lower=0.0 upper=1.5708 effort=100 velocity=100
- added joint md3_flexion_left: type revolute, parent midph3_left, child distph3_left, origin xyz=-0.0015679045780434622 -0.033364779691156365 0.0022444582750893206 rpy=0.0 0.0 0.0, axis 0.9999999999999999 0.0 -1.1075375161486551e-18, limit lower=0.0 upper=1.5708 effort=100 velocity=100
- added joint md4_flexion_left: type revolute, parent midph4_left, child distph4_left, origin xyz=0.0016320439711825516 -0.028473836326094792 -0.002199495880604859 rpy=-4.462365316954919e-33 0.19999970947446855 -1.3781457552156878e-33, axis -5.254894459090136e-16 -3.28052241842023e-33 -1.0000000000000007, limit lower=0.0 upper=1.5708 effort=100 velocity=100
- added joint md5_flexion_left: type revolute, parent midph5_left, child distph5_left, origin xyz=-0.000264351531066514 -0.023750595575241493 -0.004176520440067239 rpy=0.20638367854381948 0.2682608800927275 -0.08747994233519726, axis -3.067053893791756e-16 3.6436868920186926e-17 -1.0000000000000002, limit lower=0.0 upper=1.5708 effort=100 velocity=100
- added joint mp_flexion_left: type revolute, parent firstmc_left, child proximal_thumb_left, origin xyz=-0.031296392286403026 -0.015313902373446445 -0.021977175552854895 rpy=1.252742510164709 0.5549106329448805 0.3775526480844189, axis -7.360873981229693e-17 -1.0205699454745994e-16 -1.0000000000000002, limit lower=-0.785398 upper=0.698132 effort=100 velocity=100
- added joint pm2_flexion_left: type revolute, parent proxph2_left, child midph2_left, origin xyz=-0.00896380272452799 -0.04793519890568425 0.0038243567913669348 rpy=-3.1093030719372425 -1.326545003064804 2.985625911527994, axis -6.004321121326396e-16 -1.7684176337434925e-16 -0.9999999999999996, limit lower=0.0 upper=1.5708 effort=100 velocity=100
- added joint pm3_flexion_left: type revolute, parent proxph3_left, child midph3_left, origin xyz=-0.0032791804486541187 -0.050782878607970316 0.006636901655556221 rpy=0.0 -0.19999959192895989 0.0, axis 0.9999999999999999 0.0 -1.1075375161486551e-18, limit lower=0.0 upper=1.5708 effort=100 velocity=100
- added joint pm4_flexion_left: type revolute, parent proxph4_left, child midph4_left, origin xyz=0.0029770056462484693 -0.04623882695175058 0.003153798086735826 rpy=-3.141592653589793 -1.5207955451442956 -3.141592653589793, axis -1.228163387906391e-16 -2.5729218551481257e-33 -1.0000000000000002, limit lower=0.0 upper=1.5708 effort=100 velocity=100
- added joint pm5_flexion_left: type revolute, parent proxph5_left, child midph5_left, origin xyz=0.006871847516719935 -0.04084937033623416 0.0006944757577670244 rpy=0.0 -1.5707963267948961 0.0, axis 1.019142349991081e-16 0.0 -1.0000000000000004, limit lower=0.0 upper=1.5708 effort=100 velocity=100
- added joint rotate_x_joint_left: type revolute, parent joint_tz_link_left, child joint_rx_link_left, origin xyz=0 0 0 rpy=0 0 0, axis 1 0 0, limit lower=-3.141593 upper=3.141593 effort=100 velocity=100
- added joint rotate_y_joint_left: type revolute, parent joint_rx_link_left, child joint_ry_link_left, origin xyz=0 0 0 rpy=0 0 0, axis 0 1 0, limit lower=-3.141593 upper=3.141593 effort=100 velocity=100
- added joint rotate_z_joint_left: type revolute, parent joint_ry_link_left, child joint_rz_link_left, origin xyz=0 0 0 rpy=0 0 0, axis 0 0 1, limit lower=-3.141593 upper=3.141593 effort=100 velocity=100
- added joint translate_x_joint_left: type prismatic, parent world, child joint_tx_link_left, origin xyz=0 0 0 rpy=0 0 0, axis 1 0 0, limit lower=-1.0 upper=1.0 effort=20.0 velocity=5.0
- added joint translate_y_joint_left: type prismatic, parent joint_tx_link_left, child joint_ty_link_left, origin xyz=0 0 0 rpy=0 0 0, axis 0 1 0, limit lower=-1.0 upper=1.0 effort=20.0 velocity=5.0
- added joint translate_z_joint_left: type prismatic, parent joint_ty_link_left, child joint_tz_link_left, origin xyz=0 0 0 rpy=0 0 0, axis 0 0 1, limit lower=-1.0 upper=1.0 effort=20.0 velocity=5.0
- added joint wrist_fixed_left: type fixed, parent joint_rz_link_left, child lunate_left, origin xyz=0.0 0.0 0.0 rpy=0.0 0.0 0.0
- joint IFtip_joint: origin xyz=0.001807957398170786 -0.018019268531468673 0.00019300683206118223 rpy=1.5707963267948983 -1.47079632685829 -1.4707963268582915 -> xyz=0.0020767067263732755 -0.020697797526362065 0.0002216969198405811 rpy=1.5707963267948983 -1.47079632685829 -1.4707963268582915
- joint LFtip_joint: origin xyz=-0.0002639275958432456 -0.017259588011967385 0.0010183142350493565 rpy=-0.3006875686285624 -0.6985554313998293 0.11023436132302193 -> xyz=-0.00030315991633306173 -0.019825191984694294 0.0011696846527624262 rpy=-0.3006875686285624 -0.6985554313998293 0.11023436132302193
- joint MFtip_joint: origin xyz=0.002 -0.019 -0.001 rpy=0.0 0.0 0.0 -> xyz=0.002297296085045365 -0.021824312807930967 -0.0011486480425226826 rpy=0.0 0.0 0.0
- joint RFtip_joint: origin xyz=-0.001389977929764417 -0.018000000000000002 -0.00026069398682713335 rpy=0.0 -0.9707969349430002 0.0 -> xyz=-0.0015965954281736284 -0.02067566476540829 -0.0002994456376664207 rpy=0.0 -0.9707969349430002 0.0
- joint THtip_joint: origin xyz=0.009841981910666443 -0.021512696300755037 0.0020830962391582093 rpy=-0.500912540251172 0.05012299056598368 -0.012825373716091965 -> xyz=0.011304973256230661 -0.024710516495247227 0.002392744417495439 rpy=-0.500912540251172 0.05012299056598368 -0.012825373716091965
- joint capitate2fifthmc_fixed: origin xyz=-0.021896 -0.034683 -0.004218 rpy=0.0 0.0 0.0 -> xyz=-0.025150797539076657 -0.0398385600588142 -0.004844997443360676 rpy=0.0 0.0 0.0
- joint capitate2fourthmc_fixed: origin xyz=-0.012046 -0.040519 0.003513 rpy=0.0 0.0 0.0 -> xyz=-0.013836614320228233 -0.046542070034976575 0.004035200573382184 rpy=0.0 0.0 0.0
- joint capitate2hamate_fixed: origin xyz=-0.010969 -0.002495 -0.00075 rpy=0.0 0.0 0.0 -> xyz=-0.012599520378431305 -0.002865876866094093 -0.000861486031892012 rpy=0.0 0.0 0.0
- joint capitate2secondmc_fixed: origin xyz=0.014685 -0.03762 0.005032 rpy=0.0 0.0 0.0 -> xyz=0.016867896504445593 -0.04321213935970332 0.005779996949974139 rpy=0.0 0.0 0.0
- joint capitate2thirdmc_fixed: origin xyz=0.000477 -0.039239 0.007377 rpy=0.0 0.0 0.0 -> xyz=0.0005479051162833196 -0.045071800540547546 0.00847357660968983 rpy=0.0 0.0 0.0
- joint capitate2trapezium_fixed: origin xyz=0.015293 -0.004569 -0.010308 rpy=0.0 0.0 0.0 -> xyz=0.017566274514299384 -0.005248172906286137 -0.01184026402232381 rpy=0.0 0.0 0.0
- joint capitate2trapezoid_fixed: origin xyz=0.009143 -0.004062 -0.002464 rpy=0.0 0.0 0.0 -> xyz=0.010502089052784887 -0.004665808348727136 -0.00283026877677589 rpy=0.0 0.0 0.0
- joint cmc_abduction: origin xyz=0.0072 -0.0054 -0.0025 rpy=0.7286789533902661 -0.042411704128519245 -0.01617642349516324 -> xyz=0.008270265906163315 -0.006202699429622487 -0.0028716201063067066 rpy=0.7286789533902661 -0.042411704128519245 -0.01617642349516324
- joint ip_flexion: origin xyz=0.01332315574203723 -0.0275339009948909 -0.0057617546873297495 rpy=0.2947943417533358 0.032709979997034955 -0.01102290149135593 -> xyz=0.015303616763315903 -0.031626761480794775 -0.006618228243097208 rpy=0.2947943417533358 0.032709979997034955 -0.01102290149135593
- joint lunate2capitate_fixed: origin xyz=0.003992 -0.015054 0.002327 rpy=0.0 0.0 0.0 -> xyz=0.004585402985750549 -0.017291747632136464 0.0026729039949502827 rpy=0.0 0.0 0.0
- joint lunate2pisiform_fixed: origin xyz=-0.013388 -0.009886 -0.010593 rpy=0.0 0.0 0.0 -> xyz=-0.015378099993293676 -0.011355534548379242 -0.012167628714442777 rpy=0.0 0.0 0.0
- joint lunate2scaphoid_fixed: origin xyz=0.012345 -0.004464 -0.001254 rpy=0.0 0.0 0.0 -> xyz=0.014180060084942516 -0.005127564861821255 -0.001440404645323444 rpy=0.0 0.0 0.0
- joint lunate2triquetrum_fixed: origin xyz=-0.010784 -0.007499 -0.001289 rpy=0.0 0.0 0.0 -> xyz=-0.01238702049056461 -0.008613711670877596 -0.001480607326811738 rpy=0.0 0.0 0.0
- joint mcp2_flexion: origin xyz=0.003501 -0.028243 0.00362 rpy=-1.5707963267948977 1.4708802086674053 -1.4708802086674064 -> xyz=0.004021416796871912 -0.032441266664968126 0.004158105913932111 rpy=-1.5707963267948977 1.4708802086674053 -1.4708802086674064
- joint mcp3_flexion: origin xyz=0.00024 -0.02629 0.001778 rpy=0.0 1.370796734865936 0.0 -> xyz=0.0002756755302054438 -0.030197957037921327 0.00204229621960533 rpy=0.0 1.370796734865936 0.0
- joint mcp4_flexion: origin xyz=-0.00183 -0.023689 -0.000173 rpy=0.0 1.1207958627668684 0.0 -> xyz=-0.002102025917816509 -0.02721032347931983 -0.0001987161113564241 rpy=0.0 1.1207958627668684 0.0
- joint mcp5_flexion: origin xyz=-0.001597 -0.021431 -0.001496 rpy=0.0 0.9707969349430003 0.0 -> xyz=-0.001834390923908724 -0.02461667619930361 -0.0017183774716139331 rpy=0.0 0.9707969349430003 0.0
- joint md2_flexion: origin xyz=0.0012127706679736369 -0.02510505928504355 0.0005244221594777518 rpy=0.0221383296958119 -0.1977786936551691 2.5098334244206405e-05 -> xyz=0.0013930466537968441 -0.02883687720518117 0.0006023764869396378 rpy=0.0221383296958119 -0.1977786936551691 2.5098334244206405e-05
- joint md3_flexion: origin xyz=0.001365 -0.029047 0.001954 rpy=0.0 0.0 0.0 -> xyz=0.0015679045780434616 -0.03336477969115636 0.002244458275089322 rpy=0.0 0.0 0.0
- joint md4_flexion: origin xyz=-0.001420839030551271 -0.024789 -0.00191485624767556 rpy=0.0 -0.199999709474469 0.0 -> xyz=-0.0016320439711825436 -0.02847383632609478 -0.002199495880604861 rpy=0.0 -0.199999709474469 0.0
- joint md5_flexion: origin xyz=0.0002301414543709532 -0.020677000000000004 -0.0036360314782713345 rpy=0.20638367854381953 -0.26826088009272797 0.08747994233519721 -> xyz=0.0002643515310665187 -0.023750595575241513 -0.004176520440067224 rpy=0.20638367854381953 -0.26826088009272797 0.08747994233519721
- joint mp_flexion: origin xyz=0.027246285309179025 -0.013332110277934892 -0.019133080577570315 rpy=1.2527425101647096 -0.5549106329448805 -0.37755264808441874 -> xyz=0.03129639228640301 -0.015313902373446452 -0.0219771755528549 rpy=1.2527425101647096 -0.5549106329448805 -0.37755264808441874
- joint pm2_flexion: origin xyz=0.007803785313420723 -0.041731842245086755 0.0033294417870314806 rpy=-3.1093030719372434 1.3265450030648043 -2.985625911527994 -> xyz=0.008963802724527972 -0.04793519890568429 0.0038243567913669326 rpy=-3.1093030719372434 1.3265450030648043 -2.985625911527994
- joint pm3_flexion: origin xyz=0.002854817426452336 -0.044211 0.005778011549107881 rpy=0.0 0.1999995919289601 0.0 -> xyz=0.0032791804486541182 -0.05078287860797032 0.006636901655556221 rpy=0.0 0.1999995919289601 0.0
- joint pm4_flexion: origin xyz=-0.0025917474596572772 -0.040255 0.0027456609596525293 rpy=3.141592653589793 1.5207955451442956 3.141592653589793 -> xyz=-0.0029770056462484666 -0.046238826951750585 0.003153798086735828 rpy=3.141592653589793 1.5207955451442956 3.141592653589793
- joint pm5_flexion: origin xyz=-0.005982552759701617 -0.035563 0.0006046027434494238 rpy=-0.0 1.5707963267948966 0.0 -> xyz=-0.0068718475167199354 -0.04084937033623416 0.0006944757577670242 rpy=-0.0 1.5707963267948966 0.0
