Commit message: Update the joint limits of wrist joints

File: configs/urdfs/myohand_two_scaled.urdf (robot description, URDF)
Before this commit: robot myohand_two_scaled, 87 links, 86 joints
Joints:
- joint translate_x_joint: limit lower=-1.0 upper=1.0 effort=20.0 velocity=5.0 -> lower=-10.0 upper=10.0 effort=20.0 velocity=5.0
- joint translate_x_joint_left: limit lower=-1.0 upper=1.0 effort=20.0 velocity=5.0 -> lower=-10.0 upper=10.0 effort=20.0 velocity=5.0
- joint translate_y_joint: limit lower=-1.0 upper=1.0 effort=20.0 velocity=5.0 -> lower=-10.0 upper=10.0 effort=20.0 velocity=5.0
- joint translate_y_joint_left: limit lower=-1.0 upper=1.0 effort=20.0 velocity=5.0 -> lower=-10.0 upper=10.0 effort=20.0 velocity=5.0
- joint translate_z_joint: limit lower=-1.0 upper=1.0 effort=20.0 velocity=5.0 -> lower=-10.0 upper=10.0 effort=20.0 velocity=5.0
- joint translate_z_joint_left: limit lower=-1.0 upper=1.0 effort=20.0 velocity=5.0 -> lower=-10.0 upper=10.0 effort=20.0 velocity=5.0
