Commit message: Add the myohand for Elizabeth

File: configs/urdfs/myohand_two_scaled_ruocheng.urdf (robot description, URDF)
Before this commit: robot myohand_two_scaled, 81 links, 80 joints
Links:
- link capitate: geometry visual mesh filename=package://myohand_description/meshes/capitate.stl scale=1.0912156403965485 1.0912156403965485 1.0912156403965485
- link capitate_left: geometry visual mesh filename=package://myohand_description/meshes/capitate_left.stl scale=1.0912156403965485 1.0912156403965485 1.0912156403965485
- link distal_thumb: geometry collision cylinder length=0.023732372288272855 radius=0.007092901662577565; collision sphere radius=0.007092901662577565
- link distal_thumb_left: geometry collision cylinder length=0.023732372288272855 radius=0.007092901662577565; collision sphere radius=0.007092901662577565
- link distph2: geometry collision cylinder length=0.017459450246344776 radius=0.00763850948277584; collision sphere radius=0.00763850948277584
- link distph2_left: geometry collision cylinder length=0.017459450246344776 radius=0.00763850948277584; collision sphere radius=0.00763850948277584
- link distph3: geometry collision cylinder length=0.017459450246344776 radius=0.00763850948277584; collision sphere radius=0.00763850948277584
- link distph3_left: geometry collision cylinder length=0.017459450246344776 radius=0.00763850948277584; collision sphere radius=0.00763850948277584
- link distph4: geometry collision cylinder length=0.017459450246344776 radius=0.007420266354696529; collision sphere radius=0.007420266354696529
- link distph4_left: geometry collision cylinder length=0.017459450246344776 radius=0.007420266354696529; collision sphere radius=0.007420266354696529
- link distph5: geometry collision cylinder length=0.01527701896555168 radius=0.006547293842379291; collision sphere radius=0.006547293842379291
- link distph5_left: geometry collision cylinder length=0.01527701896555168 radius=0.006547293842379291; collision sphere radius=0.006547293842379291
- link fifthmc: geometry collision cylinder length=0.05237835073903433 radius=0.01036654858376721; collision sphere radius=0.01036654858376721
- link fifthmc_left: geometry collision cylinder length=0.05237835073903433 radius=0.01036654858376721; collision sphere radius=0.01036654858376721
- link firstmc: geometry collision cylinder length=0.044872453647446034 radius=0.01036654858376721; collision sphere radius=0.01036654858376721
- link firstmc_left: geometry collision cylinder length=0.044872453647446034 radius=0.01036654858376721; collision sphere radius=0.01036654858376721
- link fourthmc: geometry collision cylinder length=0.05674321330062052 radius=0.01036654858376721; collision sphere radius=0.01036654858376721
- link fourthmc_left: geometry collision cylinder length=0.05674321330062052 radius=0.01036654858376721; collision sphere radius=0.01036654858376721
- link hamate: geometry collision sphere radius=0.004364862561586194; visual mesh filename=package://myohand_description/meshes/hamate.stl scale=1.0912156403965485 1.0912156403965485 1.0912156403965485
- link hamate_left: geometry collision sphere radius=0.004364862561586194; visual mesh filename=package://myohand_description/meshes/hamate_left.stl scale=1.0912156403965485 1.0912156403965485 1.0912156403965485
- link lunate: geometry collision sphere radius=0.0016368234605948228; collision sphere radius=0.002182431280793097
- link lunate_left: geometry collision sphere radius=0.0016368234605948228; collision sphere radius=0.002182431280793097
- link midph2: geometry collision cylinder length=0.026189175369517165 radius=0.008729725123172388; collision sphere radius=0.008729725123172388
- link midph2_left: geometry collision cylinder length=0.026189175369517165 radius=0.008729725123172388; collision sphere radius=0.008729725123172388
- link midph3: geometry collision cylinder length=0.03055403793110336 radius=0.008729725123172388; collision sphere radius=0.008729725123172388
- link midph3_left: geometry collision cylinder length=0.03055403793110336 radius=0.008729725123172388; collision sphere radius=0.008729725123172388
- link midph4: geometry collision cylinder length=0.02182431280793097 radius=0.008184117302974114; collision sphere radius=0.008184117302974114
- link midph4_left: geometry collision cylinder length=0.02182431280793097 radius=0.008184117302974114; collision sphere radius=0.008184117302974114
- link midph5: geometry collision cylinder length=0.01964188152713787 radius=0.00763850948277584; collision sphere radius=0.00763850948277584
- link midph5_left: geometry collision cylinder length=0.01964188152713787 radius=0.00763850948277584; collision sphere radius=0.00763850948277584
- link pisiform: geometry visual mesh filename=package://myohand_description/meshes/pisiform.stl scale=1.0912156403965485 1.0912156403965485 1.0912156403965485
- link pisiform_left: geometry visual mesh filename=package://myohand_description/meshes/pisiform_left.stl scale=1.0912156403965485 1.0912156403965485 1.0912156403965485
- link proximal_thumb: geometry collision cylinder length=0.03396503996425633 radius=0.009275332943370664; collision sphere radius=0.009275332943370664
- link proximal_thumb_left: geometry collision cylinder length=0.03396503996425633 radius=0.009275332943370664; collision sphere radius=0.009275332943370664
- link proxph2: geometry collision cylinder length=0.04364862561586194 radius=0.009820940763568936; collision sphere radius=0.009820940763568936
- link proxph2_left: geometry collision cylinder length=0.04364862561586194 radius=0.009820940763568936; collision sphere radius=0.009820940763568936
- link proxph3: geometry collision cylinder length=0.04801348817744813 radius=0.009820940763568936; collision sphere radius=0.009820940763568936
- link proxph3_left: geometry collision cylinder length=0.04801348817744813 radius=0.009820940763568936; collision sphere radius=0.009820940763568936
- link proxph4: geometry collision cylinder length=0.03928376305427574 radius=0.009275332943370664; collision sphere radius=0.009275332943370664
- link proxph4_left: geometry collision cylinder length=0.03928376305427574 radius=0.009275332943370664; collision sphere radius=0.009275332943370664
- link proxph5: geometry collision cylinder length=0.03491890049268955 radius=0.008729725123172388; collision sphere radius=0.008729725123172388
- link proxph5_left: geometry collision cylinder length=0.03491890049268955 radius=0.008729725123172388; collision sphere radius=0.008729725123172388
- link scaphoid: geometry visual mesh filename=package://myohand_description/meshes/scaphoid.stl scale=1.0912156403965485 1.0912156403965485 1.0912156403965485
- link scaphoid_left: geometry visual mesh filename=package://myohand_description/meshes/scaphoid_left.stl scale=1.0912156403965485 1.0912156403965485 1.0912156403965485
- link secondmc: geometry collision cylinder length=0.06110807586220672 radius=0.010912156403965485; collision sphere radius=0.010912156403965485
- link secondmc_left: geometry collision cylinder length=0.06110807586220672 radius=0.010912156403965485; collision sphere radius=0.010912156403965485
- link thirdmc: geometry collision cylinder length=0.06110807586220672 radius=0.010912156403965485; collision sphere radius=0.010912156403965485
- link thirdmc_left: geometry collision cylinder length=0.06110807586220672 radius=0.010912156403965485; collision sphere radius=0.010912156403965485
- link trapezium: geometry collision sphere radius=0.012003372044362033; visual mesh filename=package://myohand_description/meshes/trapezium.stl scale=1.0912156403965485 1.0912156403965485 1.0912156403965485
- link trapezium_left: geometry collision sphere radius=0.012003372044362033; visual mesh filename=package://myohand_description/meshes/trapezium_left.stl scale=1.0912156403965485 1.0912156403965485 1.0912156403965485
- link trapezoid: geometry visual mesh filename=package://myohand_description/meshes/trapezoid.stl scale=1.0912156403965485 1.0912156403965485 1.0912156403965485
- link trapezoid_left: geometry visual mesh filename=package://myohand_description/meshes/trapezoid_left.stl scale=1.0912156403965485 1.0912156403965485 1.0912156403965485
- link triquetrum: geometry visual mesh filename=package://myohand_description/meshes/triquetrum.stl scale=1.0912156403965485 1.0912156403965485 1.0912156403965485
- link triquetrum_left: geometry visual mesh filename=package://myohand_description/meshes/triquetrum_left.stl scale=1.0912156403965485 1.0912156403965485 1.0912156403965485
Joints:
- joint IFtip_joint: origin xyz=0.0017859677846810168 -0.017800105872671373 0.0001906593510628998 rpy=1.5707963267948983 -1.47079632685829 -1.4707963268582915 -> xyz=0.001972871390054612 -0.01966290765004396 0.00021061207384855205 rpy=1.5707963267948983 -1.47079632685829 -1.4707963268582915
- joint IFtip_joint_left: origin xyz=-0.001785967784681018 -0.017800105872671383 -0.00019065935106290198 rpy=-1.5707963267948983 -1.47079632685829 1.4707963268582915 -> xyz=-0.0019728713900546107 -0.019662907650043953 -0.00021061207384855162 rpy=-1.5707963267948983 -1.47079632685829 1.4707963268582915
- joint LFtip_joint: origin xyz=-0.0002607175280464331 -0.017049665106837093 0.0010059288013756855 rpy=-0.3006875686285624 -0.6985554313998293 0.11023436132302193 -> xyz=-0.0002880019205164087 -0.018833932385459582 0.0011112004201243048 rpy=-0.3006875686285624 -0.6985554313998293 0.11023436132302193
- joint LFtip_joint_left: origin xyz=0.010492417503838123 -0.013441288212440073 -0.001005928801375686 rpy=2.8409050849612303 -0.6985554313998293 -2.3532617678330627 -> xyz=0.011590461196100244 -0.014847934653276816 -0.0011112004201243 rpy=2.8409050849612303 -0.6985554313998293 -2.3532617678330627
- joint MFtip_joint: origin xyz=0.001975674633139014 -0.01876890901482063 -0.000987837316569507 rpy=0.0 0.0 0.0 -> xyz=0.002182431280793097 -0.02073309716753442 -0.0010912156403965485 rpy=0.0 0.0 0.0
- joint MFtip_joint_left: origin xyz=-0.0019756746331390145 -0.018768909014820645 -0.0009878373165695085 rpy=0.0 0.0 0.0 -> xyz=-0.0021824312807930974 -0.02073309716753441 -0.0010912156403965478 rpy=0.0 0.0 0.0
- joint RFtip_joint: origin xyz=-0.0013730720682293206 -0.017781071698251126 -0.0002575232483931218 rpy=0.0 -0.9707969349430002 0.0 -> xyz=-0.0015167656567649471 -0.019641881527137875 -0.0002844733557830997 rpy=0.0 -0.9707969349430002 0.0
- joint RFtip_joint_left: origin xyz=-0.0013730720682293219 -0.017781071698251133 0.0002575232483931224 rpy=3.141592653589793 -0.970796934943 3.141592653589793 -> xyz=-0.0015167656567649462 -0.01964188152713786 0.00028447335578309926 rpy=3.141592653589793 -0.970796934943 3.141592653589793
- joint THtip_joint: origin xyz=0.009722277000358368 -0.021251044185912615 0.002057760199046078 rpy=-0.500912540251172 0.05012299056598368 -0.012825373716091965 -> xyz=0.010739724593419127 -0.02347499067048487 0.0022731071966206693 rpy=-0.500912540251172 0.05012299056598368 -0.012825373716091965
- joint THtip_joint_left: origin xyz=-0.013904280259131693 0.018782985373439132 -0.0020577601990460805 rpy=2.6406801133386213 0.05012299056598368 0.19534205721336395 -> xyz=-0.015359379356017569 0.0207486466334502 -0.002273107196620666 rpy=2.6406801133386213 0.05012299056598368 0.19534205721336395
- joint capitate2fifthmc_fixed: origin xyz=-0.021629685883605924 -0.034261161650580206 -0.0041666978012901805 rpy=0.0 0.0 0.0 -> xyz=-0.023893257662122826 -0.03784663205587349 -0.004602747571192642 rpy=0.0 0.0 0.0
- joint capitate2fifthmc_fixed_left: origin xyz=0.021629685883605924 -0.034261161650580206 -0.0041666978012901805 rpy=0.0 0.0 0.0 -> xyz=0.023893257662122826 -0.03784663205587349 -0.004602747571192642 rpy=0.0 0.0 0.0
- joint capitate2fourthmc_fixed: origin xyz=-0.01189948831539628 -0.04002618023007985 0.003470272493108678 rpy=0.0 0.0 0.0 -> xyz=-0.013144783604216823 -0.04421496653322775 0.003833440544713075 rpy=0.0 0.0 0.0
- joint capitate2fourthmc_fixed_left: origin xyz=0.011899488315396282 -0.04002618023007985 0.003470272493108678 rpy=0.0 0.0 0.0 -> xyz=0.013144783604216823 -0.04421496653322775 0.003833440544713075 rpy=0.0 0.0 0.0
- joint capitate2hamate_fixed: origin xyz=-0.010835587525450921 -0.0024646541048409195 -0.0007408779874271302 rpy=0.0 0.0 0.0 -> xyz=-0.01196954435950974 -0.002722583022789388 -0.0008184117302974114 rpy=0.0 0.0 0.0
- joint capitate2hamate_fixed_left: origin xyz=0.010835587525450921 -0.002464654104840919 -0.0007408779874271301 rpy=0.0 0.0 0.0 -> xyz=0.01196954435950974 -0.002722583022789389 -0.0008184117302974113 rpy=0.0 0.0 0.0
- joint capitate2secondmc_fixed: origin xyz=0.014506390993823209 -0.03716243984934485 0.004970797376977759 rpy=0.0 0.0 0.0 -> xyz=0.016024501679223317 -0.04105153239171815 0.005490997102475432 rpy=0.0 0.0 0.0
- joint capitate2secondmc_fixed_left: origin xyz=-0.014506390993823209 -0.03716243984934485 0.004970797376977759 rpy=0.0 0.0 0.0 -> xyz=-0.016024501679223317 -0.04105153239171815 0.005490997102475432 rpy=0.0 0.0 0.0
- joint capitate2thirdmc_fixed: origin xyz=0.0004711984000036548 -0.038761748464870883 0.007287275884333253 rpy=0.0 0.0 0.0 -> xyz=0.0005205098604691537 -0.04281821051352017 0.008049897779205338 rpy=0.0 0.0 0.0
- joint capitate2thirdmc_fixed_left: origin xyz=-0.00047119840000365513 -0.038761748464870883 0.007287275884333253 rpy=0.0 0.0 0.0 -> xyz=-0.000520509860469154 -0.04281821051352017 0.008049897779205338 rpy=0.0 0.0 0.0
- joint capitate2trapezium_fixed: origin xyz=0.015106996082297468 -0.004513428699406077 -0.010182627059198477 rpy=0.0 0.0 0.0 -> xyz=0.016687960788584415 -0.00498576426097183 -0.01124825082120762 rpy=0.0 0.0 0.0
- joint capitate2trapezium_fixed_left: origin xyz=-0.015106996082297468 -0.004513428699406076 -0.010182627059198476 rpy=0.0 0.0 0.0 -> xyz=-0.016687960788584415 -0.004985764260971831 -0.01124825082120762 rpy=0.0 0.0 0.0
- joint capitate2trapezoid_fixed: origin xyz=0.009031796585395001 -0.004012595179905337 -0.002434031148027265 rpy=0.0 0.0 0.0 -> xyz=0.009976984600145643 -0.004432517931290779 -0.0026887553379370955 rpy=0.0 0.0 0.0
- joint capitate2trapezoid_fixed_left: origin xyz=-0.009031796585395001 -0.004012595179905336 -0.002434031148027265 rpy=0.0 0.0 0.0 -> xyz=-0.009976984600145643 -0.0044325179312907775 -0.0026887553379370955 rpy=0.0 0.0 0.0
- joint cmc_abduction: origin xyz=0.00711242867930045 -0.005334321509475337 -0.0024695932914237675 rpy=0.7286789533902661 -0.042411704128519245 -0.01617642349516324 -> xyz=0.00785675261085515 -0.005892564458141362 -0.0027280391009913713 rpy=0.7286789533902661 -0.042411704128519245 -0.01617642349516324
- joint cmc_abduction_left: origin xyz=-0.00711242867930045 -0.005334321509475336 -0.002469593291423768 rpy=-2.4129137001995273 -0.042411704128519245 0.11111240339895034 -> xyz=-0.00785675261085515 -0.005892564458141361 -0.0027280391009913713 rpy=-2.4129137001995273 -0.042411704128519245 0.11111240339895034
- joint ip_flexion: origin xyz=0.013161110416451675 -0.0271990148734835 -0.005691676289063598 rpy=0.2947943417533358 0.032709979997034955 -0.01102290149135593 -> xyz=0.014538435925150106 -0.030045423406755034 -0.006287316830942347 rpy=0.2947943417533358 0.032709979997034955 -0.01102290149135593
- joint ip_flexion_left: origin xyz=-0.028539543656225103 0.009924499250664028 0.0056916762890635965 rpy=0.2822749386733923 0.09214204995112318 0.5745146568145356 -> xyz=-0.03152624008536495 0.010963109637361421 0.006287316830942348 rpy=0.2822749386733923 0.09214204995112318 0.5745146568145356
- joint lunate2capitate_fixed: origin xyz=0.003943446567745471 -0.014870902963637357 0.0022986974356572426 rpy=0.0 0.0 0.0 -> xyz=0.004356132836463022 -0.016427160250529642 0.0025392587952027686 rpy=0.0 0.0 0.0
- joint lunate2capitate_fixed_left: origin xyz=-0.003943446567745471 -0.014870902963637357 0.0022986974356572426 rpy=0.0 0.0 0.0 -> xyz=-0.004356132836463022 -0.016427160250529642 0.0025392587952027686 rpy=0.0 0.0 0.0
- joint lunate2pisiform_fixed: origin xyz=-0.01322516599423256 -0.009765759711606146 -0.010464160694420787 rpy=0.0 0.0 0.0 -> xyz=-0.014609194993628992 -0.01078775782096028 -0.011559247278720639 rpy=0.0 0.0 0.0
- joint lunate2pisiform_fixed_left: origin xyz=0.01322516599423256 -0.009765759711606146 -0.010464160694420787 rpy=0.0 0.0 0.0 -> xyz=0.014609194993628992 -0.01078775782096028 -0.011559247278720639 rpy=0.0 0.0 0.0
- joint lunate2scaphoid_fixed: origin xyz=0.012194851673050563 -0.004409705781166279 -0.0012387479949781616 rpy=0.0 0.0 0.0 -> xyz=0.013471057080695391 -0.0048711866187301925 -0.0013683844130572718 rpy=0.0 0.0 0.0
- joint lunate2scaphoid_fixed_left: origin xyz=-0.012194851673050563 -0.004409705781166279 -0.0012387479949781616 rpy=0.0 0.0 0.0 -> xyz=-0.013471057080695391 -0.0048711866187301925 -0.0013683844130572718 rpy=0.0 0.0 0.0
- joint lunate2triquetrum_fixed: origin xyz=-0.010652837621885562 -0.007407792036954732 -0.0012733223010580944 rpy=0.0 0.0 0.0 -> xyz=-0.01176766946603638 -0.008183026087333716 -0.001406576960471151 rpy=0.0 0.0 0.0
- joint lunate2triquetrum_fixed_left: origin xyz=0.010652837621885562 -0.007407792036954732 -0.0012733223010580944 rpy=0.0 0.0 0.0 -> xyz=0.01176766946603638 -0.008183026087333716 -0.001406576960471151 rpy=0.0 0.0 0.0
- joint mcp2_flexion: origin xyz=0.0034584184453098437 -0.027899489331872585 0.003575971085981615 rpy=-1.5707963267948977 1.4708802086674053 -1.4708802086674064 -> xyz=0.0038203459570283166 -0.03081920333171972 0.003950200618235505 rpy=-1.5707963267948977 1.4708802086674053 -1.4708802086674064
- joint mcp2_flexion_left: origin xyz=-0.0034584184453098424 -0.027899489331872585 0.0035759710859816158 rpy=1.5707963267948977 1.4708802086674053 1.4708802086674064 -> xyz=-0.003820345957028317 -0.030819203331719724 0.003950200618235505 rpy=1.5707963267948977 1.4708802086674053 1.4708802086674064
- joint mcp3_flexion: origin xyz=0.00023708095597668166 -0.02597024305261234 0.0017563747488605834 rpy=0.0 1.370796734865936 0.0 -> xyz=0.00026189175369517164 -0.02868805918602526 0.0019401814086250633 rpy=0.0 1.370796734865936 0.0
- joint mcp3_flexion_left: origin xyz=-0.00023708095597668125 -0.025970243052612342 0.0017563747488605827 rpy=-3.141592653589793 1.3707967348659365 3.141592653589793 -> xyz=-0.0002618917536951716 -0.028688059186025267 0.0019401814086250635 rpy=-3.141592653589793 1.3707967348659365 3.141592653589793
- joint mcp4_flexion: origin xyz=-0.0018077422893221977 -0.02340087819221505 -0.0001708958557665247 rpy=0.0 1.1207958627668684 0.0 -> xyz=-0.001996924621925684 -0.02584980730535384 -0.0001887803057886029 rpy=0.0 1.1207958627668684 0.0
- joint mcp4_flexion_left: origin xyz=0.0018077422893221975 -0.02340087819221505 -0.00017089585576652438 rpy=-3.141592653589793 1.1207958627668684 3.141592653589793 -> xyz=0.0019969246219256834 -0.025849807305353835 -0.00018878030578860314 rpy=-3.141592653589793 1.1207958627668684 3.141592653589793
- joint mcp5_flexion: origin xyz=-0.0015775761945615023 -0.021170341531401102 -0.0014778046255879823 rpy=0.0 0.9707969349430003 0.0 -> xyz=-0.0017426713777132878 -0.02338584238933843 -0.0016324585980332365 rpy=0.0 0.9707969349430003 0.0
- joint mcp5_flexion_left: origin xyz=0.001577576194561503 -0.021170341531401106 -0.0014778046255879826 rpy=-3.141592653589793 0.9707969349430003 3.141592653589793 -> xyz=0.001742671377713289 -0.023385842389338433 -0.0016324585980332365 rpy=-3.141592653589793 0.9707969349430003 3.141592653589793
- joint md2_flexion: origin xyz=0.001198020122265286 -0.024799714396455806 0.0005180437787680879 rpy=0.0221383296958119 -0.1977786936551691 2.5098334244206405e-05 -> xyz=0.0013233943211070024 -0.027395033344922118 0.0005722576625926557 rpy=0.0221383296958119 -0.1977786936551691 2.5098334244206405e-05
- joint md2_flexion_left: origin xyz=-0.003851925448209623 -0.024528019828362925 -0.0005180437787680853 rpy=0.018120226299812726 0.19818193015538843 -1.6818641285691258e-05 -> xyz=-0.004255033925347842 -0.027094905624354404 -0.0005722576625926579 rpy=0.018120226299812726 0.19818193015538843 -1.6818641285691258e-05
- joint md3_flexion: origin xyz=0.0013483979371173768 -0.028693710534394467 0.0019302341165768164 rpy=0.0 0.0 0.0 -> xyz=0.0014895093491412886 -0.031696540706598546 0.002132235361334856 rpy=0.0 0.0 0.0
- joint md3_flexion_left: origin xyz=-0.001348397937117377 -0.02869371053439447 0.001930234116576817 rpy=0.0 0.0 0.0 -> xyz=-0.001489509349141288 -0.03169654070659855 0.0021322353613348576 rpy=0.0 0.0 0.0
- joint md4_flexion: origin xyz=-0.0014035578152169872 -0.024487499240441506 -0.0018915664573201801 rpy=0.0 -0.199999709474469 0.0 -> xyz=-0.0015504417726234165 -0.027050144509790038 -0.0020895210865746177 rpy=0.0 -0.199999709474469 0.0
- joint md4_flexion_left: origin xyz=-0.001403557815216987 -0.024487499240441496 0.0018915664573201805 rpy=4.865991258798914e-17 0.19999970947446966 -2.2559491645940666e-16 -> xyz=-0.0015504417726234152 -0.02705014450979004 0.002089521086574618 rpy=4.865991258798914e-17 0.19999970947446966 -2.2559491645940666e-16
- joint md5_flexion: origin xyz=0.00022734231671720574 -0.020425512194707698 -0.0035918075784578123 rpy=0.20638367854381953 -0.26826088009272797 0.08747994233519721 -> xyz=0.0002511339545131927 -0.022563065796479438 -0.003967694418063864 rpy=0.20638367854381953 -0.26826088009272797 0.08747994233519721
- joint md5_flexion_left: origin xyz=0.00022734231671720442 -0.0204255121947077 0.0035918075784578136 rpy=-0.3270437039190569 0.08255811450688944 -0.5762987939281994 -> xyz=0.00025113395451319235 -0.022563065796479445 0.003967694418063864 rpy=-0.3270437039190569 0.08255811450688944 -0.5762987939281994
- joint mp_flexion: origin xyz=0.02691489736630659 -0.013169956041163946 -0.018900370975455213 rpy=1.2527425101647096 -0.5549106329448805 -0.37755264808441874 -> xyz=0.029731572672082863 -0.01454820725477413 -0.02087831677521216 rpy=1.2527425101647096 -0.5549106329448805 -0.37755264808441874
- joint mp_flexion_left: origin xyz=-0.022218378662445786 -0.02010480270923298 0.01890037097545521 rpy=1.296173942622059 0.1996933528297966 0.5854313730048055 -> xyz=-0.024543557824794764 -0.022208793690431786 0.020878316775212156 rpy=1.296173942622059 0.1996933528297966 0.5854313730048055
- joint pm2_flexion: origin xyz=0.0077088703430940545 -0.04122427105888849 0.0032889468405755606 rpy=-3.1093030719372434 1.3265450030648043 -2.985625911527994 -> xyz=0.008515612588301573 -0.045538438960400086 0.003633138951798585 rpy=-3.1093030719372434 1.3265450030648043 -2.985625911527994
- joint pm2_flexion_left: origin xyz=0.03421474263602158 0.024253218191698858 -0.003288946840575564 rpy=-2.4780393093699837 -1.258961676197502 -1.7039987731665693 -> xyz=0.037795355237465696 0.026791345676876653 -0.0036331389517985876 rpy=-2.4780393093699837 -1.258961676197502 -1.7039987731665693
- joint pm3_flexion: origin xyz=0.0028200951858425413 -0.04367327560285447 0.005707735423778349 rpy=0.0 0.1999995919289601 0.0 -> xyz=0.0031152214262214124 -0.04824373467757181 0.00630505657277841 rpy=0.0 0.1999995919289601 0.0
- joint pm3_flexion_left: origin xyz=0.002820095185842542 -0.04367327560285447 -0.0057077354237783495 rpy=3.141592653589793 0.19999959192896033 3.141592653589793 -> xyz=0.0031152214262214132 -0.048243734677571815 -0.0063050565727784105 rpy=3.141592653589793 0.19999959192896033 3.141592653589793
- joint pm4_flexion: origin xyz=-0.002560224855773681 -0.0397653911785055 0.0027122663545928118 rpy=3.141592653589793 1.5207955451442956 3.141592653589793 -> xyz=-0.002828155363936044 -0.04392688560416306 0.0029961081823990368 rpy=3.141592653589793 1.5207955451442956 3.141592653589793
- joint pm4_flexion_left: origin xyz=-0.0025602248557736805 -0.0397653911785055 -0.0027122663545928126 rpy=3.141592653589791 -1.5207955451442945 -3.141592653589791 -> xyz=-0.0028281553639360442 -0.043926885604163066 -0.002996108182399038 rpy=3.141592653589791 -1.5207955451442945 -3.141592653589791
- joint pm5_flexion: origin xyz=-0.005909788864379144 -0.035130458489161374 0.0005972491516796409 rpy=-0.0 1.5707963267948966 0.0 -> xyz=-0.006528255140883939 -0.03880690181942245 0.0006597519698786732 rpy=-0.0 1.5707963267948966 0.0
- joint pm5_flexion_left: origin xyz=-0.0059097888643791455 -0.03513045848916138 -0.0005972491516796414 rpy=-5.331598161240296e-17 -1.5707963267948963 0.0 -> xyz=-0.00652825514088394 -0.03880690181942245 -0.0006597519698786737 rpy=-5.331598161240296e-17 -1.5707963267948963 0.0
